Commit message: Subido robot corregido

File: Modelo_2/Simulacion/Modelo1/urdf/Modelo1.urdf (robot description, URDF)
Before this commit: robot unnamed, 9 links, 8 joints
Links:
- link Pata_Alta_I_link: geometry collision mesh filename=../meshes/stl/Pata_Alta_I.stl scale=0.00100 0.00100 0.00100; visual mesh filename=../meshes/stl/Pata_Alta_I.stl scale=0.00100 0.00100 0.00100
Joints:
- joint Nexo_Pata_D_link_joint: origin xyz=-0.00404 -0.17761 0.00407 rpy=0.00000 0.00000 0.00000 -> xyz=-0.00404 -0.17761 0.00407 rpy=-0.00000 0.00000 -0.00000
- joint Nexo_Pata_I_link_joint: origin xyz=0.00351 -0.17611 -0.00696 rpy=0.00000 0.00000 0.00000 -> xyz=0.00351 -0.17611 -0.00696 rpy=-0.00000 0.00000 -0.00000
- joint Pata_Baja_D_link_joint: origin xyz=-0.00954 0.02939 -0.00223 rpy=0.00000 0.00000 0.00000 -> xyz=-0.00954 0.02939 -0.00223 rpy=-0.00000 0.00000 -0.00000
- joint Pata_Baja_I_link_joint: origin xyz=0.01089 0.03634 -0.00185 rpy=0.00000 0.00000 0.00000 -> xyz=0.01089 0.03634 -0.00185 rpy=-0.00000 0.00000 -0.00000

Commit message: Añadir robot

File: Modelo_2/Simulacion/Modelo1/urdf/Modelo1.urdf (robot description, URDF)
Before this commit: robot Modelo1, 9 links, 8 joints
Links:
- link Pata_Baja_D_link: mass 0.10000 -> 0.30000
- link Pata_Baja_I_link: mass 0.10000 -> 0.30000
Joints:
- joint Nexo_Pata_D_link_joint: origin xyz=-0.00404 -0.17761 0.00407 rpy=-0.00000 0.00000 -0.00000 -> xyz=-0.00404 -0.17761 0.00407 rpy=0.00000 0.00000 0.00000
- joint Nexo_Pata_I_link_joint: origin xyz=0.00351 -0.17611 -0.00696 rpy=-0.00000 0.00000 -0.00000 -> xyz=0.00351 -0.17611 -0.00696 rpy=0.00000 0.00000 0.00000
- joint Pata_Baja_D_link_joint: origin xyz=-0.00954 0.02939 -0.00223 rpy=-0.00000 0.00000 -0.00000 -> xyz=-0.00954 0.02939 -0.00223 rpy=0.00000 0.00000 0.00000
- joint Pata_Baja_I_link_joint: origin xyz=0.01089 0.03634 -0.00185 rpy=-0.00000 0.00000 -0.00000 -> xyz=0.01089 0.03634 -0.00185 rpy=0.00000 0.00000 0.00000
- joint Transversal_link_joint: limit lower=-3.14000 upper=3.14000 effort=0.00000 velocity=0.00000 -> effort=0.00000 velocity=0.00000; type revolute -> continuous
