Commit message: corrijo los pesos en el .blend

File: Modelo_3/simulacion/robot/urdf/robot.urdf (robot description, URDF)
Before this commit: robot robot, 7 links, 6 joints
Links:
- link mi_diseño-Soporte_link: mass 0.10000 -> 0.20000
- link mi_diseño-base_giratoria_link: mass 0.15000 -> 0.13000
- link mi_diseño-cuerpo001_link: mass 0.70000 -> 0.50000
- link mi_diseño-motor_soporte_d_link: mass 0.10000 -> 0.03200
- link mi_diseño-motor_soporte_i_link: mass 0.10000 -> 0.03200
- link mi_diseño-pata_d_link: mass 0.10000 -> 0.06500
- link mi_diseño-pata_i_link: mass 0.10000 -> 0.06500
Joints:
- joint mi_diseño-Soporte_link_joint: axis 0.00000 0.00000 1.00000 -> (none); limit effort=0.00000 velocity=0.00000 -> (none); type continuous -> fixed
